File: PCB/KiCad/PMT_FPGA_PCB/PMT_FPGA_PCB.kicad_pcb (KiCad board)
At the start: 2 copper layers, 3 parts, among them J1 Conn_02x20_Odd_Even, J2 Conn_01x14, J3 Conn_01x14

Commit message: firmware ok
Parts:
- removed J2, J3: Conn_01x14, Connector_PinSocket_2.54mm:PinSocket_1x14_P2.54mm_Vertical
- added C1: 10u, Capacitor_SMD:C_1206_3216Metric_Pad1.33x1.80mm_HandSolder, B.Cu at (166.4, 78.7)
- added C10: 100n, Capacitor_SMD:C_0603_1608Metric_Pad1.08x0.95mm_HandSolder, F.Cu at (155.4, 70.6)
- added C11: 10u, Capacitor_SMD:C_1206_3216Metric_Pad1.33x1.80mm_HandSolder, F.Cu at (155.4, 68.3)
- added C12: 10u, Capacitor_SMD:C_1206_3216Metric_Pad1.33x1.80mm_HandSolder, F.Cu at (154.7, 76.7)
- added C13: 100p, Capacitor_SMD:C_0603_1608Metric_Pad1.08x0.95mm_HandSolder, F.Cu at (169.9, 87.7)
- added C14: 100n, Capacitor_SMD:C_0603_1608Metric_Pad1.08x0.95mm_HandSolder, B.Cu at (166.6, 85.3)
- added C15: 100n, Capacitor_SMD:C_0603_1608Metric_Pad1.08x0.95mm_HandSolder, B.Cu at (166.6, 87.9)
- added C16: 100n, Capacitor_SMD:C_0603_1608Metric_Pad1.08x0.95mm_HandSolder, B.Cu at (154.8, 89.9)
- added C17: 100n, Capacitor_SMD:C_0603_1608Metric_Pad1.08x0.95mm_HandSolder, B.Cu at (154.8, 92.4)
- added C18: 100n, Capacitor_SMD:C_0603_1608Metric_Pad1.08x0.95mm_HandSolder, F.Cu at (179.8, 85.6)
- added C19: 100n, Capacitor_SMD:C_0603_1608Metric_Pad1.08x0.95mm_HandSolder, B.Cu at (167.1, 80.8)
- added C20: 10u, Capacitor_SMD:C_1206_3216Metric_Pad1.33x1.80mm_HandSolder, F.Cu at (179.8, 87.6)
- added C5: 100n, Capacitor_SMD:C_0603_1608Metric_Pad1.08x0.95mm_HandSolder, F.Cu at (167.6, 80.0)
- added C6: 10u, Capacitor_SMD:C_1206_3216Metric_Pad1.33x1.80mm_HandSolder, F.Cu at (165.6, 78.7)
- added C7: 100n, Capacitor_SMD:C_0603_1608Metric_Pad1.08x0.95mm_HandSolder, F.Cu at (162.4, 80.3)
- added C8: 100n, Capacitor_SMD:C_0603_1608Metric_Pad1.08x0.95mm_HandSolder, F.Cu at (162.4, 77.2)
- added C9: 100n, Capacitor_SMD:C_0603_1608Metric_Pad1.08x0.95mm_HandSolder, F.Cu at (153.9, 74.7)
- added IC1: OPA695IDBVR, opa695:SOT95P280X145-6N, F.Cu at (154.9, 91.2)
- added IC2: OPA656NB_250, KiCad_opa656:SOT95P280X145-5N, F.Cu at (166.6, 86.6)
- added IC3: AD9201ARSZ, ad9201:SOP65P777X198-28N, F.Cu at (175.3, 79.2)
- added J11: Conn_01x03, Connector_PinHeader_2.54mm:PinHeader_1x03_P2.54mm_Horizontal, F.Cu at (162.3, 63.3)
- added J13: Conn_01x02, Connector_PinHeader_2.54mm:PinHeader_1x02_P2.54mm_Vertical, B.Cu at (181.4, 112.5)
- added J4: Conn_01x03, Connector_PinHeader_2.54mm:PinHeader_1x03_P2.54mm_Vertical, B.Cu at (159.9, 74.7)
- added J5: 5449692-1, Library:TE_5449692-1, F.Cu at (144.8, 88.4)
- added J6: 5449692-1, Library:TE_5449692-1, F.Cu at (171.7, 111.5)
- added J7: 5449692-1, Library:TE_5449692-1, F.Cu at (146.9, 111.5)
- added Q1: 2N7000, Package_TO_SOT_THT:TO-92_Inline, B.Cu at (173.3, 89.1)
- added R1: 5k, Resistor_SMD:R_0805_2012Metric_Pad1.20x1.40mm_HandSolder, F.Cu at (155.4, 72.6)
- added R10: 50, Resistor_SMD:R_0805_2012Metric_Pad1.20x1.40mm_HandSolder, F.Cu at (144.3, 107.2)
- added R11: 50, Resistor_SMD:R_0805_2012Metric_Pad1.20x1.40mm_HandSolder, F.Cu at (169.4, 107.2)
- added R12: Y, Resistor_SMD:R_0805_2012Metric_Pad1.20x1.40mm_HandSolder, F.Cu at (164.6, 70.4)
- added R13: X, Resistor_SMD:R_0805_2012Metric_Pad1.20x1.40mm_HandSolder, F.Cu at (164.6, 74.3)
- added R2: PVG5A101C03R00, PVG5A101C03R00:TRIM_PVG5A101C03R00, F.Cu at (159.1, 86.5)
- added R3: 50, Resistor_SMD:R_0805_2012Metric_Pad1.20x1.40mm_HandSolder, F.Cu at (149.1, 86.1)
- added R4: 470, Resistor_SMD:R_0805_2012Metric_Pad1.20x1.40mm_HandSolder, F.Cu at (158.2, 91.2)
- added R6: 47k, Resistor_SMD:R_0805_2012Metric_Pad1.20x1.40mm_HandSolder, F.Cu at (151.6, 91.2)
- added R8: 110, Resistor_SMD:R_0805_2012Metric_Pad1.20x1.40mm_HandSolder, F.Cu at (162.2, 89.9)
- added R9: 100, Resistor_SMD:R_0805_2012Metric_Pad1.20x1.40mm_HandSolder, F.Cu at (163.3, 85.1)
- added REF**: MountingHole_3.2mm_M3, MountingHole:MountingHole_3.2mm_M3, F.Cu at (145.0, 65.5)
- added RV1: 10k, Potentiometer_THT:Potentiometer_Bourns_3296Y_Vertical, B.Cu at (154.7, 78.7)
- J1: moved to B.Cu
- moved J1 116.2 mm to (187.7, 64.3), turned to 180 degrees
Connections:
- J1 pad 1: GPIO_0 -> CLOCK
- J1 pad 12: GND -> AVSS
- J1 pad 13: GPIO_10 -> D6
- J1 pad 15: GPIO_12 -> D5
- J1 pad 17: GPIO_14 -> D4
- J1 pad 19: GPIO_16 -> D3
- J1 pad 21: GPIO_18 -> D2
- J1 pad 23: GPIO_20 -> D1
- J1 pad 25: GPIO_22 -> D0
- J1 pad 30: GND -> AVSS
- J1 pad 5: GPIO_4 -> D9
- J1 pad 7: GPIO_6 -> D8
- J1 pad 9: GPIO_8 -> D7
Routing:
- net AVSS: track 0.00 -> 78.6 mm, vias 0 -> 1
- net +5V: track 0.00 -> 56.3 mm, vias 0 -> 3
- net GPIO_28: track 0.00 -> 48.7 mm
- net -5V: track 0.00 -> 40.9 mm, vias 0 -> 2
- net INB-Q: track 0.00 -> 37.7 mm
- net VREF: track 0.00 -> 23.8 mm
- net GPIO_26: track 0.00 -> 23.4 mm
- net REFSENSE: track 0.00 -> 22.8 mm
- net GPIO_30: track 0.00 -> 22.1 mm
- net 3.3V: track 0.00 -> 21.3 mm
- net D0: track 0.00 -> 17.1 mm
- net CLOCK: track 0.00 -> 15.4 mm
- net D1: track 0.00 -> 15.4 mm
- net GPIO_2: track 0.00 -> 14.6 mm
- net INA-Q: track 0.00 -> 14.5 mm
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- added copper zone on B.Cu, net (none)
- added copper zone on B.Cu, net AVSS
- added copper zone on F.Cu, net AVSS
