File: PCB/KiCad/PMT_FPGA_PCB/PMT_FPGA_PCB.kicad_sch (KiCad schematic)
At the start: 18 parts, among them J1 Conn_02x20_Odd_Even, J2 Conn_01x14, J3 Conn_01x14, J4 Conn_01x03

Commit message: firmware ok
Parts:
- removed C1, C2, C4: 100n, Capacitor_SMD:C_0201_0603Metric_Pad0.64x0.40mm_HandSolder, symbol Device:C_Small
- removed C3: 10u, Capacitor_SMD:C_1206_3216Metric_Pad1.33x1.80mm_HandSolder, symbol Device:C_Polarized_Small_US
- removed J2, J3: Conn_01x14, Connector_PinSocket_2.54mm:PinSocket_1x14_P2.54mm_Vertical, symbol Connector_Generic:Conn_01x14
- added C1, C20: 10u, Capacitor_SMD:C_1206_3216Metric_Pad1.33x1.80mm_HandSolder, symbol Device:C_Polarized_Small_US
- added C13: 100p, Capacitor_SMD:C_0603_1608Metric_Pad1.08x0.95mm_HandSolder, symbol Device:C_Small
- added C14, C15, C16, C17, C18, C19: 100n, Capacitor_SMD:C_0603_1608Metric_Pad1.08x0.95mm_HandSolder, symbol Device:C_Small
- added IC1: OPA695IDBVR, SOT95P280X145-6N, symbol OPA695IDBVR:OPA695IDBVR
- added IC2: OPA656NB_250, KiCad_opa656:SOT95P280X145-5N, symbol OPA656NB_250:OPA656NB_250
- added IC3: AD9201ARSZ, SOP65P777X198-28N, symbol AD9201ARSZ:AD9201ARSZ
- added J11: Conn_01x03, Connector_PinHeader_2.54mm:PinHeader_1x03_P2.54mm_Horizontal, symbol Connector_Generic:Conn_01x03
- added J13: Conn_01x02, Connector_PinHeader_2.54mm:PinHeader_1x02_P2.54mm_Vertical, symbol Connector_Generic:Conn_01x02
- added J5, J6, J7: 5449692-1, Library:TE_5449692-1, symbol sma-5449692-1:5449692-1
- added Q1: 2N7000, Package_TO_SOT_THT:TO-92_Inline, symbol Transistor_FET:2N7000
- added R10, R11, R3: 50, Resistor_SMD:R_0805_2012Metric_Pad1.20x1.40mm_HandSolder, symbol Device:R_Small_US
- added R12: Y, Resistor_SMD:R_0805_2012Metric_Pad1.20x1.40mm_HandSolder, symbol Device:R_Small_US
- added R13: X, Resistor_SMD:R_0805_2012Metric_Pad1.20x1.40mm_HandSolder, symbol Device:R_Small_US
- added R2: PVG5A101C03R00, PVG5A101C03R00:TRIM_PVG5A101C03R00, symbol PVG5A101C03R00:PVG5A101C03R00
- added R4: 470, Resistor_SMD:R_0805_2012Metric_Pad1.20x1.40mm_HandSolder, symbol Device:R_Small_US
- added R6: 47k, Resistor_SMD:R_0805_2012Metric_Pad1.20x1.40mm_HandSolder, symbol Device:R_Small_US
- added R8: 110, Resistor_SMD:R_0805_2012Metric_Pad1.20x1.40mm_HandSolder, symbol Device:R_Small_US
- added R9: 100, Resistor_SMD:R_0805_2012Metric_Pad1.20x1.40mm_HandSolder, symbol Device:R_Small_US
- C10, C5, C7, C8, C9: footprint Capacitor_SMD:C_0201_0603Metric_Pad0.64x0.40mm_HandSolder -> Capacitor_SMD:C_0603_1608Metric_Pad1.08x0.95mm_HandSolder
- RV1: footprint Potentiometer_THT:Potentiometer_Bourns_3296W_Vertical -> Potentiometer_THT:Potentiometer_Bourns_3296Y_Vertical
Connections:
- net GPIO_0 is gone; now on net CLOCK: J1.1 (Pin_1)
- net GPIO_10 is gone; now on net D6: J1.13 (Pin_13)
- net GPIO_12 is gone; now on net D5: J1.15 (Pin_15)
- net GPIO_14 is gone; now on net D4: J1.17 (Pin_17)
- net GPIO_16 is gone; now on net D3: J1.19 (Pin_19)
- net GPIO_18 is gone; now on net D2: J1.21 (Pin_21)
- net GPIO_20 is gone; now on net D1: J1.23 (Pin_23)
- net GPIO_22 is gone; now on net D0: J1.25 (Pin_25)
- net GPIO_4 is gone; now on net D9: J1.5 (Pin_5)
- net GPIO_6 is gone; now on net D8: J1.7 (Pin_7)
- net GPIO_8 is gone; now on net D7: J1.9 (Pin_9)
- net REFB_Q is gone; now on net REFB-Q: C5.2, C6.2, C8.1
- net REFT_Q is gone; now on net REFT-Q: C5.1, C6.1, C7.2
- net 3.3V: now also C18.1, C20.1, IC3.2 (DVDD)
- net CLOCK: now also IC3.14 (CLOCK)
- net D0: now also IC3.3 (D0)
- net D1: now also IC3.4 (D1)
- net D2: now also IC3.5 (D2)
- net D3: now also IC3.6 (D3)
- net D4: now also IC3.7 (D4)
- net D5: now also IC3.8 (D5)
- net D6: now also IC3.9 (D6)
- net D7: now also IC3.10 (D7)
- net D8: now also IC3.11 (D8)
- net D9: now also IC3.12 (D9)
- net GND: now also C1.2, C14.2, C15.2, C16.2, C17.2, C18.2, C19.2, C20.2, IC3.1 (DVSS), IC3.15 (SLEEP), IC3.20 (AVSS), IC3.28 (CHIP-SELECT), J11.2 (Pin_2), J5.S1, J5.S2, J6.S1, J6.S2, J7.S1, J7.S2, R10.1, R11.1, R12.1, R3.1, R6.1, R9.2
- net GPIO_2: now also IC3.13 (SELECT)
- net GPIO_26: now also Q1.2 (G)
- net GPIO_28: now also J7.1, R10.2
- net GPIO_30: now also J6.1, R11.2
- net GPIO_32: now also J13.2 (Pin_2)
- net GPIO_34: now also J13.1 (Pin_1)
- net INA-I: now also IC3.16 (INA-I)
- net INA-Q: now also C13.1, IC2.1 (V_OUT), IC3.27 (INA-Q), Q1.3 (D)
- net INB-I: now also IC3.17 (INB-I); no longer C12.1, C9.1, R1.1, RV1.1, RV1.2
- net INB-Q: now also C12.1, C9.1, R1.1, RV1.1, RV1.2, IC3.26 (INB-Q)
- net REFB-I: now also IC3.19 (REFB-I)
- net REFB-Q: now also IC3.24 (REFB-Q)
- net REFSENSE: now also IC3.21 (REFSENSE), R12.2, R13.1
- net REFT-I: now also IC3.18 (REFT-I)
- net REFT-Q: now also IC3.25 (REFT-Q)
- net VREF: now also IC3.22 (VREF), R13.2
- new net: R2.2, R2.3, R8.2
- new net: C13.2, IC2.4 (V_IN-), Q1.1 (S), R8.1
- new net: IC2.3 (V_IN+), R9.1
- new net: IC1.4 (INVERTING_INPUT), R4.1, R6.2
- new net +5V: C1.1, C15.1, C17.1, C19.1, IC1.5 (~{DIS}), IC1.6 (+V_S), IC2.5 (+V_S), IC3.23 (AVDD), J11.3 (Pin_3)
- new net -5V: C14.1, C16.1, IC1.2 (-V_S), IC2.2 (-V_S), J11.1 (Pin_1)
- new net OPA695: IC1.1 (OUTPUT), R2.1, R4.2
- new net PMT: IC1.3 (NONINVERTING_INPUT), J5.1, R3.2
Other:
- moved on the sheet: C10, C11, C12, C5, C6, C7, C8, C9, J1, J4, R1, RV1
